File: pcb/pcb_drumled/capteur.kicad_sch (KiCad schematic)
At the start: 0 parts

Commit message: pcb
Parts:
- added capteur: LSM6DSOXTR, Package_LGA:LGA-14_3x2.5mm_P0.5mm_LayoutBorder3x4y, symbol Sensor_Motion:LSM6DS3
- added connecteur_capteur: Conn_01x04_Pin, symbol Connector:Conn_01x04_Pin
Connections:
- new net: capteur.6 (GND), capteur.7 (GND)
Other:
- note added: "INUTILE"
Changed lines of the file:
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@@
 	(generator_version "9.0")
 	(paper "A4")
+	(text "INUTILE"
+		(exclude_from_sim no)
+		(at 113.538 71.374 0)
+		(effects
+			(font
+				(size 1.27 1.27)
+			)
+		)
+	)
+	(rule_area
+		(polyline
+			(pts
+				(xy 110.49 72.39) (xy 162.56 72.39) (xy 162.56 130.81) (xy 110.49 130.81)
+			)
+			(stroke
+				(width 0)
+				(type dash)
+			)
+			(fill
+				(type none)
+			)
+		)
+	)
+	(symbol
+		(lib_id "Sensor_Motion:LSM6DS3")
+		(at 132.08 92.71 0)
+		(unit 1)
+		(exclude_from_sim no)
+		(in_bom yes)
+		(on_board yes)
+		(dnp no)
+		(fields_autoplaced yes)
+		(property "Reference" "capteur"
+			(at 134.2233 107.95 0)
+			(effects
+				(font
+					(size 1.27 1.27)
+				)
+				(justify left)
+			)
+		)
+		(property "Value" "LSM6DSOXTR"
+			(at 134.2233 110.49 0)
+			(effects
+				(font
+					(size 1.27 1.27)
+				)
+				(justify left)
+			)
+		)
+		(property "Footprint" "Package_LGA:LGA-14_3x2.5mm_P0.5mm_LayoutBorder3x4y"
+			(at 121.92 110.49 0)
+			(effects
+				(font
+					(size 1.27 1.27)
+				)
+				(justify left)
+				(hide yes)
+			)
+		)
+		(property "Datasheet" "https://www.st.com/resource/en/datasheet/lsm6dsox.pdf"
+			(at 134.62 109.22 0)
+			(effects
+				(font
+					(size 1.27 1.27)
+				)
+				(hide yes)
+			)
+		)
+		(property "Description" "I2C/SPI, iNEMO inertial module: always-on 3D accelerometer and 3D gyroscope"
+			(at 132.08 92.71 0)
+			(effects
+				(font
+					(size 1.27 1.27)
+				)
+				(hide yes)
+			)
+		)
+		(pin "8"
+		)
+		(pin "9"
+		)
+		(pin "6"
+		)
+		(pin "10"
+		)
+		(pin "7"
+		)
+		(pin "11"
+		)
+		(pin "4"
+		)
+		(pin "3"
+		)
+		(pin "13"
+		)
+		(pin "14"
+		)
+		(pin "1"
+		)
+		(pin "2"
+		)
+		(pin "12"
+		)
+		(pin "5"
+		)
+		(instances
+			(project ""
+				(path "/184751cf-f963-4a20-a506-74be632dfa90/8959a03f-2769-4081-8c02-833ba022b4d2"
+					(reference "capteur")
+					(unit 1)
+				)
+			)
+		)
+	)
+	(symbol
+		(lib_id "Connector:Conn_01x04_Pin")
+		(at 76.2 45.72 0)
+		(unit 1)
+		(exclude_from_sim no)
+		(in_bom yes)
+		(on_board yes)
+		(dnp no)
+		(fields_autoplaced yes)
+		(property "Reference" "connecteur_capteur"
+			(at 76.835 38.1 0)
+			(effects
+				(font
+					(size 1.27 1.27)
+				)
+			)
+		)
+		(property "Value" "Conn_01x04_Pin"
+			(at 76.835 40.64 0)
+			(effects
+				(font
+					(size 1.27 1.27)
+				)
+			)
+		)
+		(property "Footprint" ""
+			(at 76.2 45.72 0)
+			(effects
+				(font
+					(size 1.27 1.27)
+				)
+				(hide yes)
+			)
+		)
+		(property "Datasheet" "~"
+			(at 76.2 45.72 0)
+			(effects
+				(font
+					(size 1.27 1.27)
+				)
+				(hide yes)
+			)
+		)
+		(property "Description" "Generic connector, single row, 01x04, script generated"
+			(at 76.2 45.72 0)
+			(effects
+				(font
+					(size 1.27 1.27)
+				)
+				(hide yes)
+			)
+		)
+		(pin "1"
+		)
+		(pin "2"
+		)
+		(pin "3"
+		)
+		(pin "4"
+		)
+		(instances
+			(project ""
+				(path "/184751cf-f963-4a20-a506-74be632dfa90/8959a03f-2769-4081-8c02-833ba022b4d2"
+					(reference "connecteur_capteur")
+					(unit 1)
+				)
+			)
+		)
+	)
 )

Commit message: pcb
Connections:
- net SCL: now reaches connecteur_capteur.1 (Pin_1)
- net SDA: now reaches connecteur_capteur.2 (Pin_2)
- net 3.3V: now reaches connecteur_capteur.3 (Pin_3)
- net GND: now reaches connecteur_capteur.4 (Pin_4)
Changed lines of the file:
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@@
+		)
+	)
+	(hierarchical_label "SDA"
+		(shape bidirectional)
+		(at 81.28 45.72 0)
+		(effects
+			(font
+				(size 1.27 1.27)
+			)
+			(justify left)
+		)
+	)
+	(hierarchical_label "3.3V"
+		(shape input)
+		(at 81.28 48.26 0)
+		(effects
+			(font
+				(size 1.27 1.27)
+			)
+			(justify left)
+		)
+	)
+	(hierarchical_label "GND"
+		(shape bidirectional)
+		(at 81.28 50.8 0)
+		(effects
+			(font
+				(size 1.27 1.27)
+			)
+			(justify left)
+		)
+	)
+	(hierarchical_label "SCL"
+		(shape bidirectional)
+		(at 81.28 43.18 0)
+		(effects
+			(font
+				(size 1.27 1.27)
+			)
+			(justify left)
 		)
 	)
