File: pcb/pcb_drumled/connectiques.kicad_sch (KiCad schematic)
At the start: 0 parts

Commit message: pcb
Parts:
- added Pad_neopixel_souder, Pad_souder_neopixel: TestPoint, symbol Connector:TestPoint
- added connecteur_batterie: Conn_01x02_Pin, symbol Connector:Conn_01x02_Pin
- added rgb_neopix: Conn_01x03_Pin, symbol Connector:Conn_01x03_Pin

Commit message: pcb
Connections:
- net Red: now reaches rgb_neopix.1 (Pin_1)
- net Green: now reaches rgb_neopix.2 (Pin_2)
- net Blue: now reaches rgb_neopix.3 (Pin_3)
- net GND: now reaches Pad_neopixel_souder.1
- net GND: now also connecteur_batterie.2 (Pin_2)
- net 5V: now reaches Pad_souder_neopixel.1
- net 5V: now also connecteur_batterie.1 (Pin_1)
Changed lines of the file:
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@@
 	(generator_version "9.0")
 	(paper "A4")
+	(hierarchical_label "GND"
+		(shape bidirectional)
+		(at 66.04 87.63 0)
+		(effects
+			(font
+				(size 1.27 1.27)
+			)
+			(justify left)
+		)
+	)
+	(hierarchical_label "Green"
+		(shape input)
+		(at 67.31 76.2 0)
+		(effects
+			(font
+				(size 1.27 1.27)
+			)
+			(justify left)
+		)
+	)
+	(hierarchical_label "5V"
+		(shape input)
+		(at 66.04 64.77 0)
+		(effects
+			(font
+				(size 1.27 1.27)
+			)
+			(justify left)
+		)
+	)
+	(hierarchical_label "Red"
+		(shape input)
+		(at 67.31 73.66 0)
+		(effects
+			(font
+				(size 1.27 1.27)
+			)
+			(justify left)
+		)
+	)
+	(hierarchical_label "Blue"
+		(shape input)
+		(at 67.31 78.74 0)
+		(effects
+			(font
+				(size 1.27 1.27)
+			)
+			(justify left)
+		)
+	)
+	(hierarchical_label "GND"
+		(shape bidirectional)
+		(at 67.31 107.95 0)
+		(effects
+			(font
+				(size 1.27 1.27)
+			)
+			(justify left)
+		)
+	)
+	(hierarchical_label "5V"
+		(shape output)
+		(at 67.31 105.41 0)
+		(effects
+			(font
+				(size 1.27 1.27)
+			)
+			(justify left)
+		)
+	)
 	(symbol
 		(lib_id "Connector:Conn_01x03_Pin")
