File: pcb/pcb_drumled/pcb_drumled.kicad_sch (KiCad schematic)
At the start: 1 part, among them U1 STM32G431KBTx

Commit message: pcb
Parts:
- added debug_uC: Conn_01x14_Pin, symbol Connector:Conn_01x14_Pin
Changed lines of the file:
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@@
+		)
+	)
+	(symbol
+		(lib_id "Connector:Conn_01x14_Pin")
+		(at 142.24 33.02 90)
+		(unit 1)
+		(exclude_from_sim no)
+		(in_bom yes)
+		(on_board yes)
+		(dnp no)
+		(fields_autoplaced yes)
+		(property "Reference" "debug_uC"
+			(at 143.51 35.56 90)
+			(effects
+				(font
+					(size 1.27 1.27)
+				)
+			)
+		)
+		(property "Value" "Conn_01x14_Pin"
+			(at 143.51 38.1 90)
+			(effects
+				(font
+					(size 1.27 1.27)
+				)
+			)
+		)
+		(property "Footprint" ""
+			(at 142.24 33.02 0)
+			(effects
+				(font
+					(size 1.27 1.27)
+				)
+				(hide yes)
+			)
+		)
+		(property "Datasheet" "~"
+			(at 142.24 33.02 0)
+			(effects
+				(font
+					(size 1.27 1.27)
+				)
+				(hide yes)
+			)
+		)
+		(property "Description" "Generic connector, single row, 01x14, script generated"
+			(at 142.24 33.02 0)
+			(effects
+				(font
+					(size 1.27 1.27)
+				)
+				(hide yes)
+			)
+		)
+		(pin "2"
+		)
+		(pin "5"
+		)
+		(pin "8"
+		)
+		(pin "9"
+		)
+		(pin "6"
+		)
+		(pin "1"
+		)
+		(pin "3"
+		)
+		(pin "4"
+		)
+		(pin "7"
+		)
+		(pin "13"
+		)
+		(pin "12"
+		)
+		(pin "14"
+		)
+		(pin "10"
+		)
+		(pin "11"
+		)
+		(instances
+			(project ""
+				(path "/184751cf-f963-4a20-a506-74be632dfa90"
+					(reference "debug_uC")
+					(unit 1)
+				)
+			)
 		)
 	)

Commit message: pcb
Parts:
- added C1: 1000u, symbol Device:C_Small
- added C2, C3: 100n, symbol Device:C_Small
- added H1, H2, H3, H4: MountingHole, symbol Mechanical:MountingHole
- added R1, R2: 4k7, symbol Device:R_Small
- added R3: 10k, symbol Device:R_Small
- added R4, R5, R6: 470, symbol Device:R_Small
Connections:
- net 3.3V: now reaches U1.1 (VDD)
- net 3.3V: now also U1.17 (VDD), C2.1, C3.2
- net 0: now reaches U1.14 (VSSA)
- net 0: now also U1.15 (VDDA), U1.16 (VSS), U1.32 (VSS), C1.1, C2.2, C3.1, R1.2, R2.2, R3.2
- net Blue: now reaches U1.18 (PA8)
- net Blue: now also R6.1
- net Green: now reaches U1.19 (PA9)
- net Green: now also R5.1
- net Red: now reaches U1.20 (PA10)
- net Red: now also R4.1
- net SCL: now reaches U1.23 (PA13)
- net SCL: now also R1.1
- net SDA: now reaches U1.24 (PA14)
- net SDA: now also R2.1
- net PA0: now reaches U1.5 (PA0)
- net PA0: now also R3.1
- new net 5V: C1.2
- new net CONNECTIQUES_NEOPIXEL_BATT_MC/Blue: R6.2
- new net CONNECTIQUES_NEOPIXEL_BATT_MC/Green: R5.2
- new net CONNECTIQUES_NEOPIXEL_BATT_MC/Red: R4.2
Other:
- sheet BOUTONS ports: added Bouton1, Bouton2, Switch1, Switch2, Switch3; removed none
- sheet CAPTEUR ports: added 3.3V, GND, SCL, SDA; removed none
- sheet CONNECTIQUES_NEOPIXEL_BATT_MC ports: added 5V, Blue, GND, Green, Red; removed none
- sheet REGULATEUR ports: added 3.3V, 5V, GND; removed none
- note added: "Trous de fixation"
- moved on the sheet: debug_uC

Commit message: pcb
Parts:
- removed H1, H2, H3, H4: MountingHole, symbol Mechanical:MountingHole
- removed debug_uC: Conn_01x14_Pin, symbol Connector:Conn_01x14_Pin
- added H1, H2, H3, H5: MountingHole_Pad, symbol Mechanical:MountingHole_Pad
- added J1: Conn_02x07_Odd_Even, symbol Connector_Generic:Conn_02x07_Odd_Even
Connections:
- net 0: now also H1.1, H2.1, H3.1, H5.1, J1.11 (Pin_11), J1.7 (Pin_7), J1.9 (Pin_9)
- net 3.3V: now also J1.13 (Pin_13)
- net 5V: now also J1.5 (Pin_5)
- net Blue: now also J1.6 (Pin_6)
- net Green: now also J1.10 (Pin_10)
- net Red: now also J1.14 (Pin_14)
- net SCL: now also J1.1 (Pin_1)
- net SDA: now also J1.2 (Pin_2)
- no-connect marks 0 -> 24

Commit message: pcb
Other:
- note added: "Connecteur test"
- moved on the sheet: J1
Changed lines of the file:
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@@
+		)
+	)
+	(text "Connecteur test"
+		(exclude_from_sim no)
+		(at 214.376 117.348 0)
+		(effects
+			(font
+				(size 1.27 1.27)
+			)
 		)
 	)
@@
 	)
 	(junction
-		(at 187.96 24.13)
+		(at 248.92 129.54)
 		(diameter 0)
 		(color 0 0 0 0)
@@
 	)
 	(no_connect
-		(at 185.42 39.37)
+		(at 246.38 144.78)
 	)
 	(no_connect
@@
 	)
 	(no_connect
-		(at 190.5 39.37)
+		(at 251.46 144.78)
 	)
 	(no_connect
-		(at 195.58 26.67)
+		(at 256.54 132.08)
 	)
 	(no_connect
@@
 	)
 	(no_connect
-		(at 195.58 39.37)
+		(at 256.54 144.78)
 	)
 	(no_connect
@@
 	(wire
 		(pts
-			(xy 187.96 24.13) (xy 187.96 26.67)
-		)
-		(stroke
-			(width 0)
-			(type default)
-		)
-	)
-	(wire
-		(pts
-			(xy 187.96 41.91) (xy 187.96 39.37)
+			(xy 248.92 129.54) (xy 248.92 132.08)
+		)
+		(stroke
+			(width 0)
+			(type default)
+		)
+	)
+	(wire
+		(pts
+			(xy 248.92 147.32) (xy 248.92 144.78)
 		)
 		(stroke
@@
 	(wire
 		(pts
-			(xy 187.96 20.32) (xy 187.96 24.13)
-		)
-		(stroke
-			(width 0)
-			(type default)
-		)
-	)
-	(wire
-		(pts
-			(xy 187.96 24.13) (xy 185.42 24.13)
+			(xy 248.92 125.73) (xy 248.92 129.54)
+		)
+		(stroke
+			(width 0)
+			(type default)
+		)
+	)
+	(wire
+		(pts
+			(xy 248.92 129.54) (xy 246.38 129.54)
 		)
 		(stroke
@@
 	(wire
 		(pts
-			(xy 182.88 25.4) (xy 182.88 26.67)
+			(xy 243.84 130.81) (xy 243.84 132.08)
 		)
 		(stroke
@@
 	(wire
 		(pts
-			(xy 190.5 24.13) (xy 187.96 24.13)
-		)
-		(stroke
-			(width 0)
-			(type default)
-		)
-	)
-	(wire
-		(pts
-			(xy 190.5 26.67) (xy 190.5 24.13)
-		)
-		(stroke
-			(width 0)
-			(type default)
-		)
-	)
-	(wire
-		(pts
-			(xy 198.12 41.91) (xy 198.12 39.37)
-		)
-		(stroke
-			(width 0)
-			(type default)
-		)
-	)
-	(wire
-		(pts
-			(xy 193.04 24.13) (xy 193.04 26.67)
+			(xy 251.46 129.54) (xy 248.92 129.54)
+		)
+		(stroke
+			(width 0)
+			(type default)
+		)
+	)
+	(wire
+		(pts
+			(xy 251.46 132.08) (xy 251.46 129.54)
+		)
+		(stroke
+			(width 0)
+			(type default)
+		)
+	)
+	(wire
+		(pts
+			(xy 259.08 147.32) (xy 259.08 144.78)
+		)
+		(stroke
+			(width 0)
+			(type default)
+		)
+	)
+	(wire
+		(pts
+			(xy 254 129.54) (xy 254 132.08)
 		)
 		(stroke
@@
 	(wire
 		(pts
-			(xy 182.88 39.37) (xy 182.88 41.91)
+			(xy 243.84 144.78) (xy 243.84 147.32)
 		)
 		(stroke
@@
 	(wire
 		(pts
-			(xy 198.12 24.13) (xy 198.12 26.67)
+			(xy 259.08 129.54) (xy 259.08 132.08)
 		)
 		(stroke
@@
 	(wire
 		(pts
-			(xy 193.04 41.91) (xy 193.04 39.37)
+			(xy 254 147.32) (xy 254 144.78)
 		)
 		(stroke
@@
 	(wire
 		(pts
-			(xy 185.42 24.13) (xy 185.42 26.67)
+			(xy 246.38 129.54) (xy 246.38 132.08)
 		)
 		(stroke
@@
 	(global_label "SDA"
 		(shape bidirectional)
-		(at 198.12 41.91 270)
+		(at 259.08 147.32 270)
 		(fields_autoplaced yes)
 		(effects
@@
 		)
 		(property "Intersheetrefs" "${INTERSHEET_REFS}"
-			(at 198.12 49.5746 90)
+			(at 259.08 154.9846 90)
 			(effects
 				(font
@@
 	(global_label "3.3V"
 		(shape bidirectional)
-		(at 182.88 25.4 90)
+		(at 243.84 130.81 90)
 		(fields_autoplaced yes)
 		(effects
@@
 		)
 		(property "Intersheetrefs" "${INTERSHEET_REFS}"
-			(at 182.88 17.1911 90)
+			(at 243.84 122.6011 90)
 			(effects
 				(font
@@
 	(global_label "SCL"
 		(shape bidirectional)
-		(at 198.12 24.13 90)
+		(at 259.08 129.54 90)
 		(fields_autoplaced yes)
 		(effects
@@
 		)
 		(property "Intersheetrefs" "${INTERSHEET_REFS}"
-			(at 198.12 16.5259 90)
+			(at 259.08 121.9359 90)
 			(effects
 				(font
@@
 	(global_label "5V"
 		(shape bidirectional)
-		(at 193.04 24.13 90)
+		(at 254 129.54 90)
 		(fields_autoplaced yes)
 		(effects
@@
 		)
 		(property "Intersheetrefs" "${INTERSHEET_REFS}"
-			(at 193.04 17.7354 90)
+			(at 254 123.1454 90)
 			(effects
 				(font
@@
 	(global_label "Blue"
 		(shape bidirectional)
-		(at 193.04 41.91 270)
+		(at 254 147.32 270)
 		(fields_autoplaced yes)
 		(effects
@@
 		)
 		(property "Intersheetrefs" "${INTERSHEET_REFS}"
-			(at 193.04 50.1793 90)
+			(at 254 155.5893 90)
 			(effects
 				(font
@@
 	(global_label "Green"
 		(shape bidirectional)
-		(at 187.96 41.91 270)
+		(at 248.92 147.32 270)
 		(fields_autoplaced yes)
 		(effects
@@
 		)
 		(property "Intersheetrefs" "${INTERSHEET_REFS}"
-			(at 187.96 51.3889 90)
+			(at 248.92 156.7989 90)
 			(effects
 				(font
@@
 	(global_label "Red"
 		(shape bidirectional)
-		(at 182.88 41.91 270)
+		(at 243.84 147.32 270)
 		(fields_autoplaced yes)
 		(effects
@@
 		)
 		(property "Intersheetrefs" "${INTERSHEET_REFS}"
-			(at 182.88 49.5141 90)
+			(at 243.84 154.9241 90)
 			(effects
 				(font
@@
 				(justify left)
 				(hide yes)
+			)
+		)
+	)
+	(rule_area
+		(polyline
+			(pts
+				(xy 270.51 157.48) (xy 270.51 119.38) (xy 207.01 119.38) (xy 207.01 157.48)
+			)
+			(stroke
+				(width 0)
+				(type dash)
+			)
+			(fill
+				(type none)
 			)
 		)
@@
 	(symbol
 		(lib_id "Connector_Generic:Conn_02x07_Odd_Even")
-		(at 190.5 31.75 270)
+		(at 251.46 137.16 270)
 		(unit 1)
 		(exclude_from_sim no)
@@
 		(fields_autoplaced yes)
 		(property "Reference" "J1"
-			(at 180.34 31.7499 90)
+			(at 241.3 137.1599 90)
 			(effects
 				(font
@@
 		)
 		(property "Value" "Conn_02x07_Odd_Even"
-			(at 180.34 34.2899 90)
+			(at 241.3 139.6999 90)
 			(effects
 				(font
@@
 		)
 		(property "Footprint" ""
-			(at 190.5 31.75 0)
+			(at 251.46 137.16 0)
 			(effects
 				(font
@@
 		)
 		(property "Datasheet" "~"
-			(at 190.5 31.75 0)
+			(at 251.46 137.16 0)
 			(effects
 				(font
@@
 		)
 		(property "Description" "Generic connector, double row, 02x07, odd/even pin numbering scheme (row 1 odd numbers, row 2 even numbers), script generated (kicad-library-utils/schlib/autogen/connector/)"
-			(at 190.5 31.75 0)
+			(at 251.46 137.16 0)
 			(effects
 				(font
@@
 	(symbol
 		(lib_id "Simulation_SPICE:0")
-		(at 187.96 20.32 180)
+		(at 248.92 125.73 180)
 		(unit 1)
 		(exclude_from_sim no)
@@
 		(dnp no)
 		(property "Reference" "#GND015"
-			(at 187.96 15.24 0)
+			(at 248.92 120.65 0)
 			(effects
 				(font
@@
 		)
 		(property "Value" "0"
-			(at 187.96 18.034 0)
+			(at 248.92 123.444 0)
 			(effects
 				(font
@@
 		)
 		(property "Footprint" ""
-			(at 187.96 20.32 0)
+			(at 248.92 125.73 0)
 			(effects
 				(font
@@
 		)
 		(property "Datasheet" "https://ngspice.sourceforge.io/docs/ngspice-html-manual/manual.xhtml#subsec_Circuit_elements__device"
-			(at 187.96 10.16 0)
+			(at 248.92 115.57 0)
 			(effects
 				(font
@@
 		)
 		(property "Description" "0V reference potential for simulation"
-			(at 187.96 12.7 0)
-			(effects
-				(font
+			(at 248.92 118.11 0)
+			(effects
+				(font

Commit message: pcb
Parts:
- removed R3: 10k, symbol Device:R_Small
- removed R5, R6: 470, symbol Device:R_Small
- added C4: 1000u, symbol Device:C_Small
- added R7: 300, symbol Device:R_Small
- added bouton_couleur1: SW_Push, symbol Switch:SW_Push
- added connecteur_batterie1: Conn_01x02_Pin, symbol Connector:Conn_01x02_Pin
- added connecteur_capteur1: Conn_01x04_Pin, symbol Connector:Conn_01x04_Pin
- added regulateur_vers_3.3V1: LD1117S33TR_SOT223, Package_TO_SOT_SMD:SOT-223-3_TabPin2, symbol Regulator_Linear:LD1117S33TR_SOT223
- added rgb_neopix1: Conn_01x03_Pin, symbol Connector:Conn_01x03_Pin
- added switch_on_off1: 472123020311, symbol Switch:SW_Nidec_CAS-120A1
- R4: value 470 -> 10k
Connections:
- net CONNECTIQUES_NEOPIXEL_BATT_MC/Red is gone; now on net 0: R4.2
- net 0: now also C4.1, connecteur_batterie1.2 (Pin_2), connecteur_capteur1.4 (Pin_4), regulateur_vers_3.3V1.1 (GND), rgb_neopix1.3 (Pin_3), switch_on_off1.1 (C)
- net 3.3V: now also C4.2, bouton_couleur1.2, connecteur_capteur1.3 (Pin_3), regulateur_vers_3.3V1.2 (VO)
- net 5V: now also regulateur_vers_3.3V1.3 (VI), rgb_neopix1.2 (Pin_2), switch_on_off1.3 (A)
- net PA0: now also R4.1, bouton_couleur1.1
- net SCL: now also U1.19 (PA9), connecteur_capteur1.1 (Pin_1); no longer U1.23 (PA13)
- net SDA: now also U1.2 (PF0), connecteur_capteur1.2 (Pin_2); no longer U1.24 (PA14)
- net Switch2: now also connecteur_batterie1.1 (Pin_1), switch_on_off1.2 (B)
- net RESET: now reaches U1.4 (PG10)
- net T_SWCLK: now reaches J1.8 (Pin_8)
- net T_SWCLK: now also U1.24 (PA14)
- net Blue: no longer names the net of U1.18 (PA8)
- net Blue: now also R7.1; no longer J1.6 (Pin_6)
- net Green renamed T_SWDIO
- net T_SWDIO: now also U1.23 (PA13); no longer U1.19 (PA9)
- removed net Red: J1.14 (Pin_14), R4.1, U1.20 (PA10)
- new net DATA_IN: J1.14 (Pin_14), R7.2, rgb_neopix1.1 (Pin_1)
- no-connect marks 24 -> 23
Other:
- removed sheet BOUTONS
- removed sheet CAPTEUR
- removed sheet CONNECTIQUES_NEOPIXEL_BATT_MC
- removed sheet REGULATEUR
- note added: "Batterie"
- note added: "Bouton couleur"
- note added: "Bouton on off"
- note added: "Capteur"
- note added: "Neopixel"
- note added: "Regulateur"
- moved on the sheet: R1, R2

Commit message: pcb
Connections:
- net RESET: now also J1.6 (Pin_6)
- no-connect marks 23 -> 22
Other:
- moved on the sheet: C2, C3, C4, H1, H2, H3, H5, J1, R1, R2, R4, R7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

Commit message: pcb
Parts:
- C1, C2, C3, C4: footprint (none) -> Capacitor_SMD:C_0603_1608Metric
- H1, H2, H3, H5: footprint (none) -> MountingHole:MountingHole_2.2mm_M2_Pad
- J1: footprint (none) -> Connector_IDC:IDC-Header_2x07_P2.54mm_Vertical
- R1, R2, R4, R7: footprint (none) -> Resistor_SMD:R_0603_1608Metric
- bouton_couleur1: footprint (none) -> Button_Switch_THT:SW_PUSH_6mm
- connecteur_batterie1: footprint (none) -> Connector_JST:JST_EH_B2B-EH-A_1x02_P2.50mm_Vertical
- connecteur_capteur1: footprint (none) -> Connector_PinHeader_1.00mm:PinHeader_1x04_P1.00mm_Vertical
- rgb_neopix1: footprint (none) -> Connector_JST:JST_EH_B3B-EH-A_1x03_P2.50mm_Vertical
- switch_on_off1: footprint (none) -> toggle:472123020311
Changed lines of the file:
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@@
 			)
 		)
-		(property "Footprint" ""
+		(property "Footprint" "Button_Switch_THT:SW_PUSH_6mm"
 			(at 91.44 146.05 0)
 			(effects
@@
 			)
 		)
-		(property "Footprint" ""
+		(property "Footprint" "Resistor_SMD:R_0603_1608Metric"
 			(at 179.07 81.28 0)
 			(effects
@@
 			)
 		)
-		(property "Footprint" ""
+		(property "Footprint" "MountingHole:MountingHole_2.2mm_M2_Pad"
 			(at 243.84 44.45 0)
 			(effects
@@
 			)
 		)
-		(property "Footprint" ""
+		(property "Footprint" "MountingHole:MountingHole_2.2mm_M2_Pad"
 			(at 220.98 36.83 0)
 			(effects
@@
 			)
 		)
-		(property "Footprint" ""
+		(property "Footprint" "Resistor_SMD:R_0603_1608Metric"
 			(at 81.28 151.13 0)
 			(effects
@@
 			)
 		)
-		(property "Footprint" ""
+		(property "Footprint" "toggle:472123020311"
 			(at 91.44 130.81 0)
 			(effects
@@
 			)
 		)
-		(property "Footprint" ""
+		(property "Footprint" "Connector_IDC:IDC-Header_2x07_P2.54mm_Vertical"
 			(at 248.92 135.89 0)
 			(effects
@@
 			)
 		)
-		(property "Footprint" ""
+		(property "Footprint" "Resistor_SMD:R_0603_1608Metric"
 			(at 167.64 76.2 0)
 			(effects
@@
 			)
 		)
-		(property "Footprint" ""
+		(property "Footprint" "Connector_JST:JST_EH_B3B-EH-A_1x03_P2.50mm_Vertical"
 			(at 158.75 149.86 0)
 			(effects
@@
 			)
 		)
-		(property "Footprint" ""
+		(property "Footprint" "Connector_JST:JST_EH_B2B-EH-A_1x02_P2.50mm_Vertical"
 			(at 187.96 144.78 0)
 			(effects
@@
 			)
 		)
-		(property "Footprint" ""
+		(property "Footprint" "MountingHole:MountingHole_2.2mm_M2_Pad"
 			(at 220.98 44.45 0)
 			(effects
@@
 			)
 		)
-		(property "Footprint" ""
+		(property "Footprint" "Resistor_SMD:R_0603_1608Metric"
 			(at 125.73 58.42 0)
 			(effects
@@
 			)
 		)
-		(property "Footprint" ""
+		(property "Footprint" "Connector_PinHeader_1.00mm:PinHeader_1x04_P1.00mm_Vertical"
 			(at 124.46 147.32 0)
 			(effects
@@
 			)
 		)
-		(property "Footprint" ""
+		(property "Footprint" "Capacitor_SMD:C_0603_1608Metric"
 			(at 257.81 72.39 0)
 			(effects
@@
 			)
 		)
-		(property "Footprint" ""
+		(property "Footprint" "Capacitor_SMD:C_0603_1608Metric"
 			(at 153.67 43.18 0)
 			(effects
@@
 			)
 		)
-		(property "Footprint" ""
+		(property "Footprint" "Capacitor_SMD:C_0603_1608Metric"
 			(at 257.81 102.87 0)
 			(effects
@@
 			)
 		)
-		(property "Footprint" ""
+		(property "Footprint" "Capacitor_SMD:C_0603_1608Metric"
 			(at 142.24 43.18 0)
 			(effects
@@
 			)
 		)
-		(property "Footprint" ""
+		(property "Footprint" "MountingHole:MountingHole_2.2mm_M2_Pad"
 			(at 243.84 36.83 0)
 			(effects
