File: pcb/pcb_drumled/pcb_drumled.kicad_sch (KiCad schematic)
At the start: 23 parts, among them J2 Conn_ST_STDC14, U1 STM32G431KBTx

Commit message: pcb
Parts:
- C1: value 1000u -> 10u
- C4: value 1000u -> 100u
Connections:
- net 3.3V: now also R1.2, R2.2
- net GND: no longer R1.2, R2.2
Changed lines of the file:
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@@
 	(wire
 		(pts
+			(xy 177.8 83.82) (xy 179.07 83.82)
+		)
+		(stroke
+			(width 0)
+			(type default)
+		)
+	)
+	(wire
+		(pts
 			(xy 86.36 151.13) (xy 86.36 147.32)
 		)
@@
 		)
 	)
+	(global_label "3.3V"
+		(shape input)
+		(at 177.8 83.82 180)
+		(fields_autoplaced yes)
+		(effects
+			(font
+				(size 1.27 1.27)
+			)
+			(justify right)
+		)
+		(property "Intersheetrefs" "${INTERSHEET_REFS}"
+			(at 170.7024 83.82 0)
+			(effects
+				(font
+					(size 1.27 1.27)
+				)
+				(justify right)
+				(hide yes)
+			)
+		)
+	)
 	(global_label "PA0"
 		(shape input)
@@
 		)
 	)
+	(global_label "3.3V"
+		(shape input)
+		(at 125.73 55.88 90)
+		(fields_autoplaced yes)
+		(effects
+			(font
+				(size 1.27 1.27)
+			)
+			(justify left)
+		)
+		(property "Intersheetrefs" "${INTERSHEET_REFS}"
+			(at 125.73 48.7824 90)
+			(effects
+				(font
+					(size 1.27 1.27)
+				)
+				(justify left)
+				(hide yes)
+			)
+		)
+	)
 	(global_label "TX"
 		(shape bidirectional)
@@
 	(symbol
 		(lib_id "power:GND")
-		(at 179.07 83.82 0)
-		(unit 1)
-		(exclude_from_sim no)
-		(in_bom yes)
-		(on_board yes)
-		(dnp no)
-		(fields_autoplaced yes)
-		(property "Reference" "#PWR010"
-			(at 179.07 90.17 0)
-			(effects
-				(font
-					(size 1.27 1.27)
-				)
-				(hide yes)
-			)
-		)
-		(property "Value" "GND"
-			(at 179.07 88.9 0)
-			(effects
-				(font
-					(size 1.27 1.27)
-				)
-			)
-		)
-		(property "Footprint" ""
-			(at 179.07 83.82 0)
-			(effects
-				(font
-					(size 1.27 1.27)
-				)
-				(hide yes)
-			)
-		)
-		(property "Datasheet" ""
-			(at 179.07 83.82 0)
-			(effects
-				(font
-					(size 1.27 1.27)
-				)
-				(hide yes)
-			)
-		)
-		(property "Description" "Power symbol creates a global label with name \"GND\" , ground"
-			(at 179.07 83.82 0)
-			(effects
-				(font
-					(size 1.27 1.27)
-				)
-				(hide yes)
-			)
-		)
-		(pin "1"
-		)
-		(instances
-			(project "pcb_drumled"
-				(path "/184751cf-f963-4a20-a506-74be632dfa90"
-					(reference "#PWR010")
-					(unit 1)
-				)
-			)
-		)
-	)
-	(symbol
-		(lib_id "power:GND")
 		(at 76.2 151.13 270)
 		(unit 1)
@@
 				)
 				(justify left)
-				(hide yes)
 			)
 		)
-		(property "Value" "1000u"
+		(property "Value" "10u"
 			(at 257.81 62.2362 0)
 			(effects
@@
 				)
 				(justify left)
-				(hide yes)
 			)
 		)
@@
 		(fields_autoplaced yes)
 		(property "Reference" "regulateur_vers_3.3V1"
-			(at 261.62 76.2 0)
+			(at 259.08 74.9299 90)
 			(effects
 				(font
 					(size 1.27 1.27)
 				)
+				(justify left)
 			)
 		)
 		(property "Value" "LD1117S33TR_SOT223"
-			(at 259.08 76.2 0)
+			(at 259.08 77.4699 90)
 			(effects
 				(font
 					(size 1.27 1.27)
 				)
+				(justify left)
 			)
 		)
@@
 	)
 	(symbol
-		(lib_id "power:GND")
-		(at 125.73 55.88 180)
-		(unit 1)
-		(exclude_from_sim no)
-		(in_bom yes)
-		(on_board yes)
-		(dnp no)
-		(fields_autoplaced yes)
-		(property "Reference" "#PWR017"
-			(at 125.73 49.53 0)
-			(effects
-				(font
-					(size 1.27 1.27)
-				)
-				(hide yes)
-			)
-		)
-		(property "Value" "GND"
-			(at 125.73 50.8 0)
-			(effects
-				(font
-					(size 1.27 1.27)
-				)
-			)
-		)
-		(property "Footprint" ""
-			(at 125.73 55.88 0)
-			(effects
-				(font
-					(size 1.27 1.27)
-				)
-				(hide yes)
-			)
-		)
-		(property "Datasheet" ""
-			(at 125.73 55.88 0)
-			(effects
-				(font
-					(size 1.27 1.27)
-				)
-				(hide yes)
-			)
-		)
-		(property "Description" "Power symbol creates a global label with name \"GND\" , ground"
-			(at 125.73 55.88 0)
-			(effects
-				(font
-					(size 1.27 1.27)
-				)
-				(hide yes)
-			)
-		)
-		(pin "1"
-		)
-		(instances
-			(project "pcb_drumled"
-				(path "/184751cf-f963-4a20-a506-74be632dfa90"
-					(reference "#PWR017")
-					(unit 1)
-				)
-			)
-		)
-	)
-	(symbol
 		(lib_id "Device:C_Small")
 		(at 153.67 43.18 90)
@@
 		(fields_autoplaced yes)
 		(property "Reference" "C4"
-			(at 252.73 92.7038 0)
+			(at 257.81 90.1635 0)
 			(effects
 				(font
 					(size 1.27 1.27)
 				)
-				(justify left)
+				(justify right)
 			)
 		)
-		(property "Value" "1000u"
-			(at 252.73 90.1638 0)
+		(property "Value" "100u"
+			(at 257.81 92.7035 0)
 			(effects
 				(font
 					(size 1.27 1.27)
 				)
-				(justify left)
+				(justify right)
 			)
 		)

Commit message: gerber
Parts:
- C4: value 100u -> 10u
Changed lines of the file:
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@@
 			)
 		)
-		(property "Value" "100u"
+		(property "Value" "10u"
 			(at 257.81 92.7035 0)
 			(effects
