File: pcb/pcb_drumled/_autosave-pcb_drumled.kicad_sch (KiCad schematic)
At the start: 20 parts, among them J1 Conn_02x07_Odd_Even, U1 STM32G431KBTx

Commit message: pcb_fini
Parts:
- removed J1: Conn_02x07_Odd_Even, Connector_IDC:IDC-Header_2x07_P2.54mm_Vertical, symbol Connector_Generic:Conn_02x07_Odd_Even
- added J2: Conn_ST_STDC14, Connector_PinHeader_1.27mm:PinHeader_2x07_P1.27mm_Vertical_SMD, symbol Connector:Conn_ST_STDC14
- added R3, R5: 10k, Resistor_SMD:R_0603_1608Metric, symbol Device:R_Small
- added reset1: SW_Push, Library:button, symbol Switch:SW_Push
- bouton_couleur1: footprint Button_Switch_THT:SW_PUSH_6mm -> Library:button
- rgb_neopix1: footprint Connector_JST:JST_EH_B3B-EH-A_1x03_P2.50mm_Vertical -> Connector_JST:JST_EH_S3B-EH_1x03_P2.50mm_Horizontal
Connections:
- net 3.3V: now also J2.3 (VCC), reset1.2
- net RESET: now also J2.12 (~{RST}), R3.1, reset1.1
- net T_SWCLK: now also J2.6 (JCLK/SWCLK)
- net T_SWDIO: now also J2.4 (JTMS/SWDIO)
- net RX: now reaches U1.20 (PA10)
- net RX: now also J2.13 (VCP_RX)
- net TX: now reaches U1.29 (PB6)
- net TX: now also J2.14 (VCP_TX)
- net at U1.31 (PB8): now also R5.1
- net 0 renamed GND
- net GND: now also J2.11 (GNDDetect), J2.5 (GND), J2.7 (GND), R3.2, R5.2; no longer switch_on_off1.1 (C)
- no-connect marks 22 -> 20
Other:
- note added: "Bouton RESET"
- note added: "Chez ST c'est comme ça"
- moved on the sheet: C4, H1, H2, H3, H5, regulateur_vers_3.3V1
